Commit message: passive wheels added

File: urdf/robot.urdf (robot description, URDF)
Before this commit: robot robot, 3 links, 2 joints
Links:
- added link bottom_left_wheel_passive; collision cylinder length=0.1 radius=0.1; visual cylinder length=0.1 radius=0.1
- added link bottom_right_wheel_passive; collision cylinder length=0.1 radius=0.1; visual cylinder length=0.1 radius=0.1
- added link top_left_wheel_passive; collision cylinder length=0.1 radius=0.1; visual cylinder length=0.1 radius=0.1
- added link top_right_wheel_passive; collision cylinder length=0.1 radius=0.1; visual cylinder length=0.1 radius=0.1
- link base: geometry collision box size=0.7 0.7 1.2; visual box size=0.7 0.7 1.2
- link left_wheel: geometry collision cylinder length=0.1 radius=0.1; visual cylinder length=0.1 radius=0.1
- link right_wheel: geometry collision cylinder length=0.1 radius=0.1; visual cylinder length=0.1 radius=0.1
Joints:
- added joint body_bottom_left_wheel: type revolute, parent base, child bottom_left_wheel_passive, origin xyz=-0.35 0.4 -0.600 rpy=-1.5707 0 0, axis 0 0 1, limit lower=-2.2 upper=0.7 effort=30 velocity=1.0
- added joint body_bottom_right_wheel: type revolute, parent base, child bottom_right_wheel_passive, origin xyz=-0.35 -0.4 -0.600 rpy=1.5707 0 0, axis 0 0 1, limit lower=-2.2 upper=0.7 effort=30 velocity=1.0
- added joint body_top_left_wheel: type revolute, parent base, child top_left_wheel_passive, origin xyz=0.35 0.4 -0.600 rpy=-1.5707 0 0, axis 0 0 1, limit lower=-2.2 upper=0.7 effort=30 velocity=1.0
- added joint body_top_right_wheel: type revolute, parent base, child top_right_wheel_passive, origin xyz=0.35 -0.4 -0.600 rpy=1.5707 0 0, axis 0 0 1, limit lower=-2.2 upper=0.7 effort=30 velocity=1.0
- joint body_left_wheel: origin xyz=0 0 0 rpy=0 0 0 -> xyz=0 0.40 -0.600 rpy=-1.5707 0 0
- joint body_right_wheel: origin xyz=0 0 0 rpy=0 0 0 -> xyz=0 -0.4 -0.600 rpy=1.5707 0 0

Commit message: ready for the differential plugin

File: urdf/robot.urdf (robot description, URDF)
Before this commit: robot robot, 7 links, 6 joints
Links:
- link base: mass None -> 1
- link bottom_left_wheel_passive: mass None -> 1
- link bottom_right_wheel_passive: mass None -> 1
- link left_wheel: mass None -> 1
- link right_wheel: mass None -> 1
- link top_left_wheel_passive: mass None -> 1
- link top_right_wheel_passive: mass None -> 1

Commit message: GOT the wheels working. to do: fix inertia and weights and add laserscan

File: urdf/robot.urdf (robot description, URDF)
Before this commit: robot robot, 7 links, 6 joints
Links:
- link base: mass 1 -> 3
Joints:
- joint body_bottom_left_wheel: limit lower=-2.2 upper=0.7 effort=30 velocity=1.0 -> effort=30 velocity=1.0; origin xyz=-0.35 0.4 -0.600 rpy=-1.5707 0 0 -> xyz=-0.35 0.41 -0.600 rpy=1.5707 0 0; type revolute -> continuous
- joint body_bottom_right_wheel: origin xyz=-0.35 -0.4 -0.600 rpy=1.5707 0 0 -> xyz=-0.35 -0.41 -0.600 rpy=1.5707 0 0; type revolute -> continuous
- joint body_left_wheel: origin xyz=0 0.40 -0.600 rpy=-1.5707 0 0 -> xyz=0 0.41 -0.600 rpy=1.5707 0 0; type revolute -> continuous
- joint body_right_wheel: origin xyz=0 -0.4 -0.600 rpy=1.5707 0 0 -> xyz=0 -0.41 -0.600 rpy=1.5707 0 0; type revolute -> continuous
- joint body_top_left_wheel: limit lower=-2.2 upper=0.7 effort=30 velocity=1.0 -> effort=30 velocity=1.0; origin xyz=0.35 0.4 -0.600 rpy=-1.5707 0 0 -> xyz=0.35 0.41 -0.600 rpy=1.5707 0 0; type revolute -> continuous
- joint body_top_right_wheel: origin xyz=0.35 -0.4 -0.600 rpy=1.5707 0 0 -> xyz=0.35 -0.41 -0.600 rpy=1.5707 0 0; type revolute -> continuous

Commit message: Mapped hostpital with working sensors and drives. to do: make to the robot fit through doors

File: urdf/robot.urdf (robot description, URDF)
Before this commit: robot robot, 7 links, 6 joints
Links:
- removed link base
- added link base_link, mass 3; collision box size=0.7 0.7 1.2; visual box size=0.7 0.7 1.2
Joints:
- joint body_bottom_left_wheel: parent base -> base_link
- joint body_bottom_right_wheel: parent base -> base_link
- joint body_left_wheel: parent base -> base_link
- joint body_right_wheel: parent base -> base_link
- joint body_top_left_wheel: parent base -> base_link
- joint body_top_right_wheel: parent base -> base_link

Commit message: fixed the directional issues

File: urdf/robot.urdf (robot description, URDF)
Before this commit: robot robot, 7 links, 6 joints
Joints:
- joint body_left_wheel: axis 0 0 1 -> 0 0 -1
- joint body_right_wheel: axis 0 0 1 -> 0 0 -1

Commit message: first commit

File: urdf/robot.urdf (robot description, URDF)
Before this commit: robot robot, 7 links, 6 joints
Links:
- added link camera_link
Joints:
- added joint camera_to_body: type fixed, parent base_link, child camera_link, origin xyz=0.35 0 0.650 rpy=0 1.22173 0

Commit message: added xacro parameters

File: urdf/robot.urdf (robot description, URDF)
Before this commit: robot robot, 8 links, 7 joints
Links:
- link base_link: geometry collision box size=${body_length} ${body_width} ${body_height}; visual box size=${body_length} ${body_width} ${body_height}
- link bottom_left_wheel_passive: geometry collision cylinder length=${wheel_thickness} radius=${wheel_diameter}; visual cylinder length=${wheel_thickness} radius=${wheel_diameter}
- link bottom_right_wheel_passive: geometry collision cylinder length=${wheel_thickness} radius=${wheel_diameter}; visual cylinder length=${wheel_thickness} radius=${wheel_diameter}
- link left_wheel: geometry collision cylinder length=${wheel_thickness} radius=${wheel_diameter}; visual cylinder length=${wheel_thickness} radius=${wheel_diameter}
- link right_wheel: geometry collision cylinder length=${wheel_thickness} radius=${wheel_diameter}; visual cylinder length=${wheel_thickness} radius=${wheel_diameter}
- link top_left_wheel_passive: geometry collision cylinder length=${wheel_thickness} radius=${wheel_diameter}; visual cylinder length=${wheel_thickness} radius=${wheel_diameter}
- link top_right_wheel_passive: geometry collision cylinder length=${wheel_thickness} radius=${wheel_diameter}; visual cylinder length=${wheel_thickness} radius=${wheel_diameter}
Joints:
- joint body_bottom_left_wheel: origin xyz=-0.35 0.41 -0.600 rpy=1.5707 0 0 -> xyz=-${body_length/2} ${body_width/2+gap+wheel_thickness/2} -${body_height/2} rpy=1.5707 0 0
- joint body_bottom_right_wheel: origin xyz=-0.35 -0.41 -0.600 rpy=1.5707 0 0 -> xyz=-${body_length/2} -${body_width/2+gap+wheel_thickness/2} -${body_height/2} rpy=1.5707 0 0
- joint body_left_wheel: origin xyz=0 0.41 -0.600 rpy=1.5707 0 0 -> xyz=0 ${body_width/2+gap+wheel_thickness/2} -${body_height/2} rpy=1.5707 0 0
- joint body_right_wheel: origin xyz=0 -0.41 -0.600 rpy=1.5707 0 0 -> xyz=0 -${body_width/2+gap+wheel_thickness/2} -${body_height/2} rpy=1.5707 0 0
- joint body_top_left_wheel: origin xyz=0.35 0.41 -0.600 rpy=1.5707 0 0 -> xyz=${body_length/2} ${body_width/2+gap+wheel_thickness/2} -${body_height/2} rpy=1.5707 0 0
- joint body_top_right_wheel: origin xyz=0.35 -0.41 -0.600 rpy=1.5707 0 0 -> xyz=${body_length/2} -${body_width/2+gap+wheel_thickness/2} -${body_height/2} rpy=1.5707 0 0

Commit message: girst ccommit

File: urdf/robot.urdf (robot description, URDF)
Before this commit: robot robot, 8 links, 7 joints
Links:
- added link laser_link
Joints:
- added joint laser_to_body: type fixed, parent base_link, child laser_link, origin xyz=0 0 ${body_height/2 + 0.01} rpy=0 0 0
